File: pcb/PCB-MTD04.kicad_sch (KiCad schematic)
At the start: 48 parts, among them J1 MotorX, J10 SC_BTNS, J2 Barrel_Jack_Switch, J3 BAU, J4 MotorY, J5 SD, J6 OLED_Screen, J7 SW_XMIN, J8 SW_YMAX, J9 SERVO, SW1 SW_Push, U1 ESP32-S3-UNO, U2 R-78E5.0-1.0

Commit message: uploadPCB
Connections:
- net +12V: now also J3.1 (Pin_1); no longer J3.2 (Pin_2)
- net +3V3: no longer A1.1 (GND), A1.7 (GND), A2.1 (GND), A2.7 (GND), C1.2, C10.2, C11.2, C12.2, C13.1, C14.2, C15.1, C16.1, C17.1, C19.2, C3.2, C4.2, C5.2, C6.2, C7.2, C8.2, C9.2, D1.1 (K), J10.5 (Pin_5), J2.2, J2.3, J5.3 (VSS), J5.6 (VSS), J6.4 (Pin_4), J7.2 (Pin_2), J8.2 (Pin_2), J9.1 (Pin_1), SW1.1, U1.29 (GND), U1.6 (GND), U1.7 (GND), U2.2 (GND)
- net at J2.1: now also J3.2 (Pin_2); no longer J3.1 (Pin_1)
- new net GND: A1.1 (GND), A1.7 (GND), A2.1 (GND), A2.7 (GND), C1.2, C10.2, C11.2, C12.2, C13.1, C14.2, C15.1, C16.1, C17.1, C19.2, C3.2, C4.2, C5.2, C6.2, C7.2, C8.2, C9.2, D1.1 (K), J10.5 (Pin_5), J2.2, J2.3, J5.3 (VSS), J5.6 (VSS), J6.4 (Pin_4), J7.2 (Pin_2), J8.2 (Pin_2), J9.1 (Pin_1), SW1.1, U1.29 (GND), U1.6 (GND), U1.7 (GND), U2.2 (GND)
Other:
- moved on the sheet: C14, C5, J3
