File: pcb/PCB-MTD04.kicad_pcb (KiCad board)
At the start: 2 copper layers, 53.3 x 87.8 mm, 48 parts, among them J1 MotorX, J10 SC_BTNS, J2 Barrel_Jack_Switch, J3 BAU, J4 MotorY, J5 SD, J6 OLED_Screen, J7 SW_XMIN, J8 SW_YMAX, J9 SERVO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

Commit message: UploadPCB
Routing:
- net +3V3: track 239.8 -> 257.2 mm, vias 7 -> 10
Changed lines of the file:
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@@
+	)
+	(segment
+		(start 137.3 118.5)
+		(end 134 118.5)
+		(width 0.35)
+		(layer "F.Cu")
+		(net 8)
 	)
 	(segment
@@
 	)
 	(segment
+		(start 128.8 121.6)
+		(end 128.8 119.98)
+		(width 0.35)
+		(layer "F.Cu")
+		(net 8)
+	)
+	(segment
 		(start 153.7 137.4)
 		(end 155.7 139.4)
@@
 	(segment
 		(start 128.8 125.025)
-		(end 128.8 119.98)
+		(end 128.8 121.6)
 		(width 0.35)
 		(layer "F.Cu")
@@
 	)
 	(segment
+		(start 131.1 121.6)
+		(end 131.2 121.5)
+		(width 0.35)
+		(layer "F.Cu")
+		(net 8)
+	)
+	(segment
 		(start 141 122.6)
 		(end 140.3 122.6)
@@
 	)
 	(segment
+		(start 128.8 121.6)
+		(end 131.1 121.6)
+		(width 0.35)
+		(layer "F.Cu")
+		(net 8)
+	)
+	(segment
 		(start 128.8 119.98)
 		(end 121.65 112.83)
@@
 	)
 	(via
+		(at 137.3 118.5)
+		(size 0.6)
+		(drill 0.3)
+		(layers "F.Cu" "B.Cu")
+		(net 8)
+	)
+	(via
 		(at 145.1 90.7)
 		(size 0.6)
 		(drill 0.3)
 		(layers "F.Cu" "B.Cu")
+		(net 8)
+	)
+	(via
+		(at 131.2 121.5)
+		(size 0.6)
+		(drill 0.3)
+		(layers "F.Cu" "B.Cu")
+		(net 8)
+	)
+	(via
+		(at 134 118.5)
+		(size 0.6)
+		(drill 0.3)
+		(layers "F.Cu" "B.Cu")
+		(net 8)
+	)
+	(segment
+		(start 132.3 118.5)
+		(end 132.3 115.8625)
+		(width 0.35)
+		(layer "B.Cu")
 		(net 8)
 	)
@@
 	)
 	(segment
+		(start 138.1 115.6)
+		(end 138.1 117.7)
+		(width 0.35)
+		(layer "B.Cu")
+		(net 8)
+	)
+	(segment
 		(start 142.2375 113.4)
 		(end 140.0375 115.6)
@@
 	)
 	(segment
+		(start 138.1 117.7)
+		(end 137.3 118.5)
+		(width 0.35)
+		(layer "B.Cu")
+		(net 8)
+	)
+	(segment
 		(start 138.075 110.8)
 		(end 139.175 109.7)
@@
 	)
 	(segment
+		(start 134 118.5)
+		(end 132.3 118.5)
+		(width 0.35)
+		(layer "B.Cu")
+		(net 8)
+	)
+	(segment
 		(start 138.4 91.7)
 		(end 139.4 90.7)
@@
 	)
 	(segment
+		(start 132.3 115.8625)
+		(end 131.8 115.3625)
+		(width 0.35)
+		(layer "B.Cu")
+		(net 8)
+	)
+	(segment
+		(start 132.3 120.4)
+		(end 132.3 118.5)
+		(width 0.35)
+		(layer "B.Cu")
+		(net 8)
+	)
+	(segment
 		(start 158.4 121)
 		(end 161.24 118.16)
@@
 		(width 0.35)
 		(layer "B.Cu")
+		(net 8)
+	)
+	(segment
+		(start 131.2 121.5)
+		(end 132.3 120.4)
+		(width 0.35)
+		(layer "B.Cu")
